File: Bridge_Rectifier/Bridge_Rectifier.kicad_sch (KiCad schematic)
At the start: 7 parts, among them J1 Screw_Terminal_01x02, J2 Screw_Terminal_01x02

Commit message: Correct Footprint of transformer and reduced hole size
Parts:
- removed J2: Screw_Terminal_01x02, TerminalBlock_Phoenix:TerminalBlock_Phoenix_MKDS-1,5-2_1x02_P5.00mm_Horizontal, symbol Connector:Screw_Terminal_01x02
- added H1, H2, H3, H4: MountingHole, MountingHole:MountingHole_2.1mm, symbol Mechanical:MountingHole
- added J2: Conn_01x02_Pin, Connector_PinHeader_2.00mm:PinHeader_1x02_P2.00mm_Vertical_SMD_Pin1Left, symbol Connector:Conn_01x02_Pin
- added T1: Transformer_1P_1S, Transformer_SMD:Transformer_ED8_4-Lead_10.5x8mm_P5mm, symbol Device:Transformer_1P_1S
- D1, D2, D3, D4: footprint Diode_THT:D_DO-41_SOD81_P10.16mm_Horizontal -> Diode_SMD:D_0805_2012Metric
- R1: footprint Resistor_THT:R_Axial_DIN0207_L6.3mm_D2.5mm_P10.16mm_Horizontal -> Resistor_SMD:R_0603_1608Metric_Pad0.98x0.95mm_HandSolder
Connections:
- net at D1.1 (K), D4.1 (K), R1.1: now also J2.2 (Pin_2)
- net at D2.1 (K), D2.2 (A), D3.2 (A)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: now also J2.1 (Pin_1), T1.3 (SA); no longer J1.2 (Pin_2)
- net at D1.2 (A), D3.1 (K): now also T1.4 (SB); no longer J1.1 (Pin_1)
- new net: J1.1 (Pin_1), T1.1 (AA)
- new net: J1.2 (Pin_2), T1.2 (AB)
Other:
- moved on the sheet: J1
