File: center_tapped_fullwaverectifier_with_filter/center_tapped_fullwaverectifier_with_filter.kicad_pcb (KiCad board)
At the start: 4 copper layers, 21 x 19 mm, 11 parts, among them J1 Screw_Terminal_01x02, J2 Conn_01x02_Pin, T1 Transformer_1P_SS

Commit message: Through holes changes to buried
Parts:
- moved J2 10.3 mm to (137.0, 81.9), turned to 0 degrees
Routing:
- net Net-(D1-K): track 40.9 -> 32.5 mm
- net Net-(J2-Pin_1): track 21.5 -> 27.9 mm
